File: grapto-v3w-pcb/grapto-v3w-pcb.kicad_sch (KiCad schematic)
At the start: 44 parts

Commit message: minor changes.
Parts:
- removed C? (x2): 22u, symbol Device:C
- removed JP?: SolderJumper_2_Open, symbol Jumper:SolderJumper_2_Open
- removed R?: 470, symbol Device:R
- removed R? (x2): 4.7K, symbol Device:R
- removed U?: TPS2110, symbol grapto-v3w:TPS2110
- added J?: Conn_01x06_Female, symbol Connector:Conn_01x06_Female
Connections:
- net 5V is gone; now on net VUSB: C?.1, D?.2 (A), U?.1 (VDD), U?.2 (VDD)
- net P+: now also C?.1, U?.8 (VIN)
- net PMUX_OUT: no longer C?.1, U?.8 (VIN)
- net SYSGND: no longer U?.2 (GND)
- no-connect marks 12 -> 11
Other:
- note removed: "Auto-Switch mode (DO=1, D1=0) OUT will switch from IN1 to IN2 when VSNS < 0.8V. - For R1=R1=4.7k, VSNS will be > 0.8 even at low usb voltages."
- note removed: "Current limit = 250/R_ilim = 250/470 A = 532 mA"
- note removed: "If PMUX is ommitted, short the jumper to power MCU directly from batter pack."
- note removed: "On resistance 120mOhm Assume Imax = 5OOmA (Charging + MCU operation) P=0.12*0.5^2 W=0.03W Dissipated heat=30/3.87C=7.75C"
- moved on the sheet: F?, J?, JP?, R?, TP?, U?
