File: grapto-v3w-pcb/grapto-v3w-pcb.kicad_pcb (KiCad board)
At the start: 2 copper layers, 145 x 73 mm, 216 parts, among them J1 Conn_01x06_Female, J2 USB_C_Receptacle_USB2.0, J3 USB_C_Receptacle_USB2.0, J4 Conn_01x06_Male, J5 Conn_01x06_Female, J6 USB_C_Receptacle_USB2.0, J7 USB_C_Receptacle_USB2.0, J8 Conn_01x06_Male, U1 AP9211S-AL, U10 MAX17260TFDN, U11 USBLC6-4SC6, U12 ACN52840, U13 TPS2110, U14 LM3676SD-3.3, U2 MCP7383x-2xMC, U3 MAX17260TFDN, U4 USBLC6-4SC6, U5 ACN52840, U6 TPS2110, U7 LM3676SD-3.3, U8 AP9211S-AL, U9 MCP7383x-2xMC

Commit message: Began case rework.
Parts:
- moved SW2 228.2 mm to (313.5, 145.8)
- moved SW15 149.9 mm to (235.5, 43.8)
- moved SW54 144.7 mm to (69.3, 160.5)
- moved SW53 141.9 mm to (171.3, 220.2)
- moved SW14 135.5 mm to (272.5, 88.8)
- moved SW32 124.3 mm to (63.5, 145.8)
- moved SW22 123.6 mm to (90.5, 77.7)
- moved SW52 101.3 mm to (185.5, 145.7)
- moved SW24 101.2 mm to (205.7, 220.2)
- moved SW46 100.3 mm to (185.5, 127.7)
- moved SW47 95.3 mm to (90.5, 131.7)
- moved SW43 95.1 mm to (128.5, 104.7)
- moved SW41 94.9 mm to (90.5, 113.7)
- moved SW51 94.8 mm to (166.5, 145.7)
- moved SW35 93.8 mm to (90.5, 95.7)
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Changed lines of the file:
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@@
     (thickness 1.6)
   )
-  (paper "A4")
+  (paper "A3")
   (layers
     (0 "F.Cu" signal)
@@
     )
     (pad_to_mask_clearance 0)
-    (grid_origin 85.45 153.97)
+    (grid_origin 13.45 199.97)
     (pcbplotparams
       (layerselection 0x00010fc_ffffffff)
@@
   )
   (footprint "Switch_Keyboard_Kailh:SW_Kailh_Choc_V1_1.00u" (layer "F.Cu")
-    (at 85.45 137.82)
+    (at 313.500 145.820 0.000)
     (descr "Kailh Choc keyswitch CPG1350 V1 with 1.00u keycap")
     (tags "Kailh Choc Keyswitch Switch CPG1350 V1 Cutout 1.00u")
@@
   )
   (footprint "Switch_Keyboard_Kailh:SW_Kailh_Choc_V1_1.00u" (layer "F.Cu")
-    (at 85.45 40.41)
+    (at 147.453 73.731)
     (descr "Kailh Choc keyswitch CPG1350 V1 with 1.00u keycap")
     (tags "Kailh Choc Keyswitch Switch CPG1350 V1 Cutout 1.00u")
@@
   )
   (footprint "Switch_Keyboard_Kailh:SW_Kailh_Choc_V1_1.00u" (layer "F.Cu")
-    (at 150.05 72.71)
+    (at 109.453 91.731)
     (descr "Kailh Choc keyswitch CPG1350 V1 with 1.00u keycap")
     (tags "Kailh Choc Keyswitch Switch CPG1350 V1 Cutout 1.00u")
@@
   )
   (footprint "Switch_Keyboard_Kailh:SW_Kailh_Choc_V1_1.00u" (layer "F.Cu")
-    (at 101.6 40.41)
+    (at 128.453 122.731)
     (descr "Kailh Choc keyswitch CPG1350 V1 with 1.00u keycap")
     (tags "Kailh Choc Keyswitch Switch CPG1350 V1 Cutout 1.00u")
@@
   )
   (footprint "Switch_Keyboard_Kailh:SW_Kailh_Choc_V1_1.00u" (layer "F.Cu")
-    (at 182.35 40.41)
+    (at 166.453 109.731)
     (descr "Kailh Choc keyswitch CPG1350 V1 with 1.00u keycap")
     (tags "Kailh Choc Keyswitch Switch CPG1350 V1 Cutout 1.00u")
@@
   )
   (footprint "Switch_Keyboard_Kailh:SW_Kailh_Choc_V1_1.00u" (layer "F.Cu")
-    (at 198.5 40.41)
+    (at 128.453 104.731)
     (descr "Kailh Choc keyswitch CPG1350 V1 with 1.00u keycap")
     (tags "Kailh Choc Keyswitch Switch CPG1350 V1 Cutout 1.00u")
@@
   )
   (footprint "Switch_Keyboard_Kailh:SW_Kailh_Choc_V1_1.00u" (layer "F.Cu")
-    (at 150.05 56.56)
+    (at 63.500 145.820 0.000)
     (descr "Kailh Choc keyswitch CPG1350 V1 with 1.00u keycap")
     (tags "Kailh Choc Keyswitch Switch CPG1350 V1 Cutout 1.00u")
@@
   )
   (footprint "Switch_Keyboard_Kailh:SW_Kailh_Choc_V1_1.00u" (layer "F.Cu")
-    (at 85.45 88.86)
+    (at 89.724 151.768)
     (descr "Kailh Choc keyswitch CPG1350 V1 with 1.00u keycap")
     (tags "Kailh Choc Keyswitch Switch CPG1350 V1 Cutout 1.00u")
@@
   )
   (footprint "Switch_Keyboard_Kailh:SW_Kailh_Choc_V1_1.00u" (layer "F.Cu")
-    (at 117.75 88.86)
+    (at 171.287 220.227 0.000)
     (descr "Kailh Choc keyswitch CPG1350 V1 with 1.00u keycap")
     (tags "Kailh Choc Keyswitch Switch CPG1350 V1 Cutout 1.00u")
@@
   )
   (footprint "Switch_Keyboard_Kailh:SW_Kailh_Choc_V1_1.00u" (layer "F.Cu")
-    (at 117.75 170.12)
+    (at 205.713 220.227 0.000)
     (descr "Kailh Choc keyswitch CPG1350 V1 with 1.00u keycap")
     (tags "Kailh Choc Keyswitch Switch CPG1350 V1 Cutout 1.00u")
@@
   )
   (footprint "Switch_Keyboard_Kailh:SW_Kailh_Choc_V1_1.00u" (layer "F.Cu")
-    (at 117.75 56.56)
+    (at 147.453 127.731)
     (descr "Kailh Choc keyswitch CPG1350 V1 with 1.00u keycap")
     (tags "Kailh Choc Keyswitch Switch CPG1350 V1 Cutout 1.00u")
@@
   )
   (footprint "Switch_Keyboard_Kailh:SW_Kailh_Choc_V1_1.00u" (layer "F.Cu")
-    (at 133.9 40.41)
+    (at 166.453 127.731)
     (descr "Kailh Choc keyswitch CPG1350 V1 with 1.00u keycap")
     (tags "Kailh Choc Keyswitch Switch CPG1350 V1 Cutout 1.00u")
@@
   )
   (footprint "Switch_Keyboard_Kailh:SW_Kailh_Choc_V1_1.00u" (layer "F.Cu")
-    (at 117.75 72.71)
+    (at 128.453 140.731)
     (descr "Kailh Choc keyswitch CPG1350 V1 with 1.00u keycap")
     (tags "Kailh Choc Keyswitch Switch CPG1350 V1 Cutout 1.00u")
@@
   )
   (footprint "Switch_Keyboard_Kailh:SW_Kailh_Choc_V1_1.00u" (layer "F.Cu")
-    (at 133.9 56.56)
+    (at 109.453 109.731)
     (descr "Kailh Choc keyswitch CPG1350 V1 with 1.00u keycap")
     (tags "Kailh Choc Keyswitch Switch CPG1350 V1 Cutout 1.00u")
@@
   )
   (footprint "Switch_Keyboard_Kailh:SW_Kailh_Choc_V1_1.00u" (layer "F.Cu")
-    (at 182.35 72.71)
+    (at 109.453 127.731)
     (descr "Kailh Choc keyswitch CPG1350 V1 with 1.00u keycap")
     (tags "Kailh Choc Keyswitch Switch CPG1350 V1 Cutout 1.00u")
@@
   )
   (footprint "Switch_Keyboard_Kailh:SW_Kailh_Choc_V1_1.00u" (layer "F.Cu")
-    (at 150.05 40.41)
+    (at 69.339 160.473)
     (descr "Kailh Choc keyswitch CPG1350 V1 with 1.00u keycap")
     (tags "Kailh Choc Keyswitch Switch CPG1350 V1 Cutout 1.00u")
@@
   )
   (footprint "Switch_Keyboard_Kailh:SW_Kailh_Choc_V1_1.00u" (layer "F.Cu")
-    (at 166.2 72.71)
+    (at 104.500 88.820 0.000)
     (descr "Kailh Choc keyswitch CPG1350 V1 with 1.00u keycap")
     (tags "Kailh Choc Keyswitch Switch CPG1350 V1 Cutout 1.00u")
@@
   )
   (footprint "Switch_Keyboard_Kailh:SW_Kailh_Choc_V1_1.00u" (layer "F.Cu")
-    (at 182.35 56.56)
+    (at 147.453 91.731)
     (descr "Kailh Choc keyswitch CPG1350 V1 with 1.00u keycap")
     (tags "Kailh Choc Keyswitch Switch CPG1350 V1 Cutout 1.00u")
@@
   )
   (footprint "Switch_Keyboard_Kailh:SW_Kailh_Choc_V1_1.00u" (layer "F.Cu")
-    (at 198.5 56.56)
+    (at 166.453 145.731)
     (descr "Kailh Choc keyswitch CPG1350 V1 with 1.00u keycap")
     (tags "Kailh Choc Keyswitch Switch CPG1350 V1 Cutout 1.00u")
@@
   )
   (footprint "Switch_Keyboard_Kailh:SW_Kailh_Choc_V1_1.00u" (layer "F.Cu")
-    (at 117.75 40.41)
+    (at 90.453 131.731)
     (descr "Kailh Choc keyswitch CPG1350 V1 with 1.00u keycap")
     (tags "Kailh Choc Keyswitch Switch CPG1350 V1 Cutout 1.00u")
@@
   )
   (footprint "Switch_Keyboard_Kailh:SW_Kailh_Choc_V1_1.00u" (layer "F.Cu")
-    (at 133.9 153.97)
+    (at 235.5 43.82)
     (descr "Kailh Choc keyswitch CPG1350 V1 with 1.00u keycap")
     (tags "Kailh Choc Keyswitch Switch CPG1350 V1 Cutout 1.00u")
@@
   )
   (footprint "Switch_Keyboard_Kailh:SW_Kailh_Choc_V1_1.00u" (layer "F.Cu")
-    (at 285.450 -46.030 0.000)
+    (at 272.500 88.820 0.000)
     (descr "Kailh Choc keyswitch CPG1350 V1 with 1.00u keycap")
     (tags "Kailh Choc Keyswitch Switch CPG1350 V1 Cutout 1.00u")
@@
   )
   (footprint "Switch_Keyboard_Kailh:SW_Kailh_Choc_V1_1.00u" (layer "F.Cu")
-    (at 166.2 56.56)
+    (at 90.453 113.731)
     (descr "Kailh Choc keyswitch CPG1350 V1 with 1.00u keycap")
     (tags "Kailh Choc Keyswitch Switch CPG1350 V1 Cutout 1.00u")
@@
   )
   (footprint "Switch_Keyboard_Kailh:SW_Kailh_Choc_V1_1.00u" (layer "F.Cu")
-    (at 133.9 72.71)
+    (at 147.453 109.731)
     (descr "Kailh Choc keyswitch CPG1350 V1 with 1.00u keycap")
     (tags "Kailh Choc Keyswitch Switch CPG1350 V1 Cutout 1.00u")
@@
   )
   (footprint "Switch_Keyboard_Kailh:SW_Kailh_Choc_V1_1.00u" (layer "F.Cu")
-    (at 150.05 88.86)
+    (at 147.453 145.731)
     (descr "Kailh Choc keyswitch CPG1350 V1 with 1.00u keycap")
     (tags "Kailh Choc Keyswitch Switch CPG1350 V1 Cutout 1.00u")
@@
   )
   (footprint "Switch_Keyboard_Kailh:SW_Kailh_Choc_V1_1.00u" (layer "F.Cu")
-    (at 101.6 56.56)
+    (at 90.453 77.731)
     (descr "Kailh Choc keyswitch CPG1350 V1 with 1.00u keycap")
     (tags "Kailh Choc Keyswitch Switch CPG1350 V1 Cutout 1.00u")
@@
   )
   (footprint "Switch_Keyboard_Kailh:SW_Kailh_Choc_V1_1.00u" (layer "F.Cu")
-    (at 166.2 88.86)
+    (at 166.453 91.731)
     (descr "Kailh Choc keyswitch CPG1350 V1 with 1.00u keycap")
     (tags "Kailh Choc Keyswitch Switch CPG1350 V1 Cutout 1.00u")
@@
   )
   (footprint "Switch_Keyboard_Kailh:SW_Kailh_Choc_V1_1.00u" (layer "F.Cu")
-    (at 166.2 40.41)
+    (at 90.453 95.731)
     (descr "Kailh Choc keyswitch CPG1350 V1 with 1.00u keycap")
     (tags "Kailh Choc Keyswitch Switch CPG1350 V1 Cutout 1.00u")
@@
   )
   (footprint "Switch_Keyboard_Kailh:SW_Kailh_Choc_V1_1.00u" (layer "F.Cu")
-    (at 85.45 72.71)
+    (at 109.453 145.731)
     (descr "Kailh Choc keyswitch CPG1350 V1 with 1.00u keycap")
     (tags "Kailh Choc Keyswitch Switch CPG1350 V1 Cutout 1.00u")
@@
   )
   (footprint "Switch_Keyboard_Kailh:SW_Kailh_Choc_V1_1.00u" (layer "F.Cu")
-    (at 133.9 88.86)
+    (at 128.453 86.731)
     (descr "Kailh Choc keyswitch CPG1350 V1 with 1.00u keycap")
     (tags "Kailh Choc Keyswitch Switch CPG1350 V1 Cutout 1.00u")
@@
   )
   (footprint "Switch_Keyboard_Kailh:SW_Kailh_Choc_V1_1.00u" (layer "F.Cu")
-    (at 85.45 56.56)
+    (at 109.453 73.731)
     (descr "Kailh Choc keyswitch CPG1350 V1 with 1.00u keycap")
     (tags "Kailh Choc Keyswitch Switch CPG1350 V1 Cutout 1.00u")
@@
   )
   (footprint "Switch_Keyboard_Kailh:SW_Kailh_Choc_V1_1.00u" (layer "F.Cu")
-    (at 198.5 137.82)
+    (at 90.453 77.731)
     (descr "Kailh Choc keyswitch CPG1350 V1 with 1.00u keycap")
     (tags "Kailh Choc Keyswitch Switch CPG1350 V1 Cutout 1.00u")
@@
   )
   (footprint "Switch_Keyboard_Kailh:SW_Kailh_Choc_V1_1.00u" (layer "F.Cu")
-    (at 101.6 72.71)
+    (at 185.453 127.731)
     (descr "Kailh Choc keyswitch CPG1350 V1 with 1.00u keycap")
     (tags "Kailh Choc Keyswitch Switch CPG1350 V1 Cutout 1.00u")
@@
   )
   (footprint "Switch_Keyboard_Kailh:SW_Kailh_Choc_V1_1.00u" (layer "F.Cu")
-    (at 101.6 88.86)
+    (at 185.453 145.731)
     (descr "Kailh Choc keyswitch CPG1350 V1 with 1.00u keycap")
     (tags "Kailh Choc Keyswitch Switch CPG1350 V1 Cutout 1.00u")

Commit message: flipping usbs
Parts:
- C1, C10, C11, C12, C13, C14, C15, C16, C17, C18, C2, C3, C4, C5, C6, C7, C8, C9, D1, D10, D11, D12, D13, D14, D15, D16, D17, D18, D19, D2, D20, D21, D22, D23, D24, D25, D26, D27, D28, D29, D3, D30, D31, D32, D33, D34, D35, D36, D37, D38, D39, D4, D40, D41, D42, D43, D44, D45, D46, D47, D48, D49, D5, D50, D51, D52, D53, D54, D55, D56, D57, D58, D59, D6, D60, D7, D8, D9, F1, F2, F3, F4, J1, J2, J3, J5, J6, J7, JP1, JP2, JP3, JP4, JP5, JP6, L1, L2, R1, R10, R11, R12, R13, R14, R15, R16, R17, R18, R19, R2, R20, R21, R22, R23, R24, R25, R26, R27, R28, R3, R4, R5, R6, R7, R8, R9, TP1, TP10, TP11, TP12, TP13, TP14, TP15, TP16, TP17, TP18, TP2, TP3, TP4, TP5, TP6, TP7, TP8, TP9, U1, U10, U12, U13, U14, U2, U5, U6, U7, U8, U9: moved to B.Cu
- moved J2 286.5 mm to (141.7, 252.0), turned to 180 degrees
- moved J6 274.3 mm to (165.4, 252.0), turned to 180 degrees
- moved J3 203.9 mm to (144.4, 215.9), turned to -90 degrees
- moved D1 50.3 mm to (193.9, -14.6), turned to 180 degrees
- moved D12 50.3 mm to (193.9, -21.3), turned to 180 degrees
- moved D22 50.3 mm to (193.9, -4.54), turned to 180 degrees
- moved D24 50.3 mm to (193.9, -7.89), turned to 180 degrees
- moved D25 50.3 mm to (193.9, -17.9), turned to 180 degrees
- moved D32 50.3 mm to (193.9, -43.3), turned to 180 degrees
- moved D38 50.3 mm to (193.9, -39.9), turned to 180 degrees
- moved D39 50.3 mm to (193.9, -53.3), turned to 180 degrees
- moved D43 50.3 mm to (193.9, -50.0), turned to 180 degrees
- moved D53 50.3 mm to (193.9, -33.2), turned to 180 degrees
- moved D55 50.3 mm to (193.9, -36.6), turned to 180 degrees
- moved D56 50.3 mm to (193.9, -46.6), turned to 180 degrees
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
Commit message: Fixing pcb coordinates.
Parts:
- moved J7 253.9 mm to (239.4, 197.8), turned to 90 degrees
- moved SW4 223.1 mm to (308.5, 126.8), turned to -90 degrees
- moved SW1 208.0 mm to (304.5, 183.8), turned to -90 degrees
- moved SW17 166.2 mm to (254.5, 88.8), turned to -90 degrees
- moved SW3 163.6 mm to (313.5, 145.8), turned to -90 degrees
- moved SW8 163.4 mm to (295.5, 145.8), turned to -90 degrees
- moved SW20 159.7 mm to (259.5, 145.8), turned to -90 degrees
- moved SW23 157.5 mm to (236.5, 88.8), turned to -90 degrees
- moved SW26 152.1 mm to (230.5, 216.1), turned to -90 degrees
- moved SW27 151.4 mm to (236.5, 164.8), turned to -90 degrees
- moved SW22 149.1 mm to (236.5, 107.8), turned to -90 degrees
- moved SW18 146.6 mm to (250.5, 183.8), turned to -90 degrees
- moved SW13 141.2 mm to (272.5, 164.8), turned to -90 degrees
- moved SW7 140.9 mm to (290.5, 164.8), turned to -90 degrees
- moved SW5 139.0 mm to (290.5, 107.8), turned to -90 degrees
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
Commit message: Think freecad and kicad models are synced now.
Parts:
- moved C17 114.2 mm to (138.6, 5.30)
- moved C8 114.2 mm to (138.6, 43.2)
- moved D30 114.2 mm to (218.7, 14.0)
- moved D31 114.2 mm to (218.7, -14.6)
- moved F2 114.2 mm to (134.2, 40.7)
- moved F4 114.2 mm to (134.2, 2.79)
- moved J4 114.2 mm to (144.2, 15.1)
- moved J7 114.2 mm to (352.5, 181.6)
- moved J8 114.2 mm to (144.2, -22.8)
- moved R10 114.2 mm to (134.2, 43.2)
- moved R11 114.2 mm to (157.4, 24.1)
- moved R12 114.2 mm to (138.6, 40.7)
- moved R14 114.2 mm to (127.6, 46.1)
- moved R20 114.2 mm to (148.7, -13.8)
- moved R23 114.2 mm to (148.7, -11.3)
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
Commit message: minor changes.
Parts:
- moved SW10 114.2 mm to (272.5, 107.8)
- moved SW11 114.2 mm to (272.5, 88.8)
- moved SW13 114.2 mm to (272.5, 164.8)
- moved SW14 114.2 mm to (277.5, 145.8)
- moved SW15 114.2 mm to (272.5, 126.8)
- moved SW16 114.2 mm to (254.5, 107.8)
- moved SW17 114.2 mm to (254.5, 88.8)
- moved SW19 114.2 mm to (254.5, 164.8)
- moved SW2 114.2 mm to (308.5, 164.8)
- moved SW20 114.2 mm to (259.5, 145.8)
- moved SW21 114.2 mm to (254.5, 126.8)
- moved SW22 114.2 mm to (236.5, 107.8)
- moved SW23 114.2 mm to (236.5, 88.8)
- moved SW28 114.2 mm to (241.5, 145.8)
- moved SW29 114.2 mm to (236.5, 126.8)
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
Commit message: Ready for layout.
Parts:
- moved J7 115.8 mm to (238.5, 201.7)
- moved J6 115.8 mm to (238.8, 218.7)
- moved SW1 20.3 mm to (284.2, 183.8)
- moved SW14 20.3 mm to (257.2, 145.8)
- moved SW2 20.3 mm to (288.2, 164.8)
- moved SW26 20.3 mm to (209.4, 184.7)
- moved SW3 20.3 mm to (293.2, 145.8)
- moved SW4 20.3 mm to (288.2, 126.8)
- moved SW5 20.3 mm to (270.2, 107.8)
- moved SW6 20.3 mm to (266.2, 183.8)
- moved SW7 20.3 mm to (270.2, 164.8)
- moved SW8 20.3 mm to (275.2, 145.8)
- moved SW9 20.3 mm to (270.2, 126.8)
- moved SW10 20.3 mm to (252.2, 107.8)
- moved SW11 20.3 mm to (252.2, 88.8)
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