File: grapto-v3w-pcb/grapto-v3w-pcb.kicad_pcb (KiCad board)
At the start: 2 copper layers, 145 x 73 mm, 216 parts, among them J1 Conn_01x06_Female, J2 USB_C_Receptacle_USB2.0, J3 USB_C_Receptacle_USB2.0, J4 Conn_01x06_Male, J5 Conn_01x06_Female, J6 USB_C_Receptacle_USB2.0, J7 USB_C_Receptacle_USB2.0, J8 Conn_01x06_Male, U1 AP9211S-AL, U10 MAX17260TFDN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

Commit message: Began layout
Parts:
- added mouse-bite-3mm-slot: VAL**, grapto-v3w:mouse-bite-3mm-slot, F.Cu at (178.3, 149.9)
- added mouse-bite-3mm-slot: VAL**, grapto-v3w:mouse-bite-3mm-slot, F.Cu at (178.4, 209.2)
- moved TP5 299.3 mm to (309.5, 209.8)
- moved TP8 299.3 mm to (305.4, 209.8)
- moved TP9 299.3 mm to (301.4, 209.8)
- moved TP7 280.0 mm to (325.5, 161.0)
- moved JP2 280.0 mm to (347.5, 170.8)
- moved TP4 280.0 mm to (333.7, 167.0)
- moved TP6 280.0 mm to (338.9, 171.6)
- moved C7 275.2 mm to (352.3, 213.9)
- moved R11 275.2 mm to (356.7, 213.9)
- moved R13 275.2 mm to (356.7, 216.4)
- moved R6 275.2 mm to (348.0, 213.9)
- moved R8 275.2 mm to (374.5, 203.8)
- moved R9 275.2 mm to (348.0, 216.4)
- moved JP3 274.7 mm to (315.0, 192.1)
- moved L1 274.7 mm to (309.5, 188.8)
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Other:
- board size 145 x 73 mm -> 244.5 x 149.5 mm
- board text added: "Top View"

Commit message: layout and snaps
Parts:
- U11, U3, U4: moved to B.Cu
- moved U4 18.0 mm to (155.4, 219.8), turned to 180 degrees
- turned U11 to 180 degrees
- turned U3 to 180 degrees

Commit message: Added snap supports.
Parts:
- removed mouse-bite-3mm-slot (x2): VAL**, grapto-v3w:mouse-bite-3mm-slot
- added TP19: ~, TestPoint:TestPoint_THTPad_D2.0mm_Drill1.0mm, F.Cu at (191.5, 204.0)
- added TP20: TestPoint, TestPoint:TestPoint_THTPad_D2.0mm_Drill1.0mm, F.Cu at (205.9, 187.8)
- added TP21: TestPoint, TestPoint:TestPoint_THTPad_D2.0mm_Drill1.0mm, F.Cu at (206.4, 193.3)
- added TP22: ~, TestPoint:TestPoint_THTPad_D2.0mm_Drill1.0mm, F.Cu at (163.1, 174.7)
- added TP23: TestPoint, TestPoint:TestPoint_THTPad_D2.0mm_Drill1.0mm, F.Cu at (151.8, 189.4)
- added TP24: TestPoint, TestPoint:TestPoint_THTPad_D2.0mm_Drill1.0mm, F.Cu at (150.8, 178.0)
- TP1, TP10, TP11, TP12, TP13, TP14, TP15, TP16, TP17, TP18, TP2, TP3, TP4, TP5, TP6, TP7, TP8, TP9: footprint TestPoint:TestPoint_Pad_2.0x2.0mm -> TestPoint:TestPoint_THTPad_D2.0mm_Drill1.0mm
- moved R22 226.1 mm to (151.6, 182.3)
- moved TP13 173.2 mm to (153.0, 211.8)
- moved TP16 172.2 mm to (163.3, 165.9)
- moved JP5 159.8 mm to (151.0, 214.8)
- moved TP12 157.0 mm to (157.5, 147.1)
- moved TP15 156.9 mm to (142.8, 210.1)
- moved TP17 156.1 mm to (167.0, 173.4)
- moved JP4 150.9 mm to (154.1, 148.3), turned to -90 degrees
- moved TP11 148.4 mm to (154.1, 151.5)
- moved TP18 147.7 mm to (154.5, 174.4)
- moved TP14 145.5 mm to (157.0, 214.8)
- moved L2 140.3 mm to (168.8, 169.3)
- moved TP10 140.1 mm to (154.1, 144.9)
- moved JP6 124.2 mm to (158.3, 174.4)
- moved C16 116.3 mm to (170.3, 161.9)
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Other:
- outline, holes or cut-outs redrawn
- copper layers 2 -> 4
