File: grapto-v3w-pcb/battery_management.kicad_sch (KiCad schematic)
At the start: 19 parts, among them U1 AP9211S-AL

Commit message: Fixed 3d model paths for pcb.
Parts:
- C10: renamed from C1; footprint (none) -> Fuse:Fuse_0603_1608Metric_Pad1.05x0.95mm_HandSolder
- C11: renamed from C2; footprint (none) -> Fuse:Fuse_0603_1608Metric_Pad1.05x0.95mm_HandSolder
- C12: renamed from C3; footprint (none) -> Fuse:Fuse_0603_1608Metric_Pad1.05x0.95mm_HandSolder
- C13: renamed from C4; footprint (none) -> Capacitor_SMD:C_0603_1608Metric_Pad1.08x0.95mm_HandSolder
- C14: renamed from C5; footprint (none) -> Capacitor_SMD:C_0603_1608Metric_Pad1.08x0.95mm_HandSolder
- D31: renamed from D30; footprint (none) -> LED_SMD:LED_0805_2012Metric_Pad1.15x1.40mm_HandSolder
- F3: renamed from F1; footprint (none) -> Fuse:Fuse_0603_1608Metric_Pad1.05x0.95mm_HandSolder
- JP4: renamed from JP1; footprint (none) -> Jumper:SolderJumper-2_P1.3mm_Bridged_RoundedPad1.0x1.5mm
- R15: renamed from R1; footprint (none) -> Resistor_SMD:R_0603_1608Metric_Pad0.98x0.95mm_HandSolder
- R16: renamed from R2; footprint (none) -> Resistor_SMD:R_0603_1608Metric_Pad0.98x0.95mm_HandSolder
- R17: renamed from R3; footprint (none) -> Resistor_SMD:R_0603_1608Metric_Pad0.98x0.95mm_HandSolder
- R18: renamed from R4; footprint (none) -> Resistor_SMD:R_0603_1608Metric_Pad0.98x0.95mm_HandSolder
- R19: renamed from R5; footprint (none) -> Resistor_SMD:R_0603_1608Metric_Pad0.98x0.95mm_HandSolder
- TP10: renamed from TP1; footprint (none) -> TestPoint:TestPoint_Pad_2.0x2.0mm
- TP11: renamed from TP2; footprint (none) -> TestPoint:TestPoint_Pad_2.0x2.0mm
- TP12: renamed from TP3; footprint (none) -> TestPoint:TestPoint_Pad_2.0x2.0mm
- U10: renamed from U3; value (none) -> MAX17260TFDN; footprint (none) -> Package_DFN_QFN:DFN-14-1EP_3x3mm_P0.4mm_EP1.78x2.35mm
- U8: renamed from U1; footprint (none) -> grapto-v3w:U-DFN2030-6_type_c
- U9: renamed from U2; value (none) -> MCP7383x-2xMC; footprint (none) -> Package_DFN_QFN:DFN-8-1EP_3x2mm_P0.5mm_EP1.75x1.45mm

Commit message: Added snap supports.
Parts:
- TP10, TP11, TP12: footprint TestPoint:TestPoint_Pad_2.0x2.0mm -> (none)
Changed lines of the file:
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@@
       (effects (font (size 1.27 1.27)) (justify left))
     )
-    (property "Footprint" "TestPoint:TestPoint_Pad_2.0x2.0mm" (id 2) (at 71.12 72.39 0)
+    (property "Footprint" "" (id 2) (at 71.12 72.39 0)
       (effects (font (size 1.27 1.27)) hide)
     )
@@
       (effects (font (size 1.27 1.27)) (justify left))
     )
-    (property "Footprint" "TestPoint:TestPoint_Pad_2.0x2.0mm" (id 2) (at 59.69 45.72 0)
+    (property "Footprint" "" (id 2) (at 59.69 45.72 0)
       (effects (font (size 1.27 1.27)) hide)
     )
@@
       (effects (font (size 1.27 1.27)) (justify left))
     )
-    (property "Footprint" "TestPoint:TestPoint_Pad_2.0x2.0mm" (id 2) (at 82.55 45.72 0)
-      (effects (font (size 1.27 1.27)) hide)
-    )
+    (property "Footprint" "" (id 2) (at 82.55 45.72 0)
+      (effects (font (size 1.27 1.27)) hide)
+    )

Commit message: More layout. esd chip problems.
Connections:
- net p-: now also C14.2, U10.15 (EP)
- net sysgnd: now also U9.9 (EP); no longer C14.2
- removed net chassi: U10.15 (EP), U9.9 (EP)
Changed lines of the file:
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@@
   (junction (at 188.595 60.96) (diameter 0) (color 0 0 0 0)
-  )
-  (junction (at 59.055 137.16) (diameter 0) (color 0 0 0 0)
   )
   (junction (at 84.455 56.515) (diameter 0) (color 0 0 0 0)
@@
   (no_connect (at 73.66 127))
   (no_connect (at 87.63 107.95))
-  (wire (pts (xy 59.055 137.16) (xy 59.055 151.765))
-    (stroke (width 0) (type default) (color 0 0 0 0))
-  )
   (wire (pts (xy 221.615 71.12) (xy 221.615 73.66))
     (stroke (width 0) (type default) (color 0 0 0 0))
@@
     (stroke (width 0) (type default) (color 0 0 0 0))
   )
-  (wire (pts (xy 59.055 107.95) (xy 59.055 137.16))
+  (wire (pts (xy 59.055 107.95) (xy 59.055 151.765))
+    (stroke (width 0) (type default) (color 0 0 0 0))
+  )
+  (wire (pts (xy 65.405 127) (xy 65.405 130.175))
     (stroke (width 0) (type default) (color 0 0 0 0))
   )
@@
     (stroke (width 0) (type default) (color 0 0 0 0))
   )
-  (wire (pts (xy 65.405 127) (xy 65.405 137.16))
-    (stroke (width 0) (type default) (color 0 0 0 0))
-  )
   (wire (pts (xy 110.49 68.58) (xy 110.49 72.39))
     (stroke (width 0) (type default) (color 0 0 0 0))
@@
   )
   (wire (pts (xy 228.6 83.82) (xy 228.6 87.63))
-    (stroke (width 0) (type default) (color 0 0 0 0))
-  )
-  (wire (pts (xy 65.405 137.16) (xy 59.055 137.16))
     (stroke (width 0) (type default) (color 0 0 0 0))
   )
@@
     (effects (font (size 1.27 1.27)) (justify left bottom))
   )
+  (label "p-" (at 85.09 139.7 0)
+    (effects (font (size 1.27 1.27)) (justify left bottom))
+  )
   (label "p-" (at 113.665 72.39 0)
     (effects (font (size 1.27 1.27)) (justify left bottom))
   )
+  (label "p-" (at 65.405 130.175 0)
+    (effects (font (size 1.27 1.27)) (justify left bottom))
+  )
   (label "p-" (at 109.855 112.395 0)
     (effects (font (size 1.27 1.27)) (justify left bottom))
@@
     (effects (font (size 1.27 1.27)) (justify left bottom))
   )
+  (hierarchical_label "sysgnd" (shape input) (at 212.725 85.09 270)
+    (effects (font (size 1.27 1.27)) (justify right))
+  )
   (hierarchical_label "low_batt" (shape output) (at 103.505 120.65 0)
     (effects (font (size 1.27 1.27)) (justify left))
@@
     (effects (font (size 1.27 1.27)) (justify left))
   )
-  (hierarchical_label "chassi" (shape input) (at 212.725 85.09 270)
-    (effects (font (size 1.27 1.27)) (justify right))
-  )
   (hierarchical_label "batt+" (shape input) (at 31.75 45.72 180)
     (effects (font (size 1.27 1.27)) (justify right))
@@
     (effects (font (size 1.27 1.27)) (justify right))
   )
-  (hierarchical_label "chassi" (shape input) (at 85.09 139.7 270)
-    (effects (font (size 1.27 1.27)) (justify right))
-  )

Commit message: Removing fuel gauge. Going for 2-layer board.
Parts:
- removed C13: .47u, Capacitor_SMD:C_0603_1608Metric_Pad1.08x0.95mm_HandSolder, symbol Device:C
- removed C14: .1u, Capacitor_SMD:C_0603_1608Metric_Pad1.08x0.95mm_HandSolder, symbol Device:C
- removed R19: 10m, Resistor_SMD:R_0603_1608Metric_Pad0.98x0.95mm_HandSolder, symbol Device:R
- removed U10: MAX17260TFDN, Package_DFN_QFN:DFN-14-1EP_3x3mm_P0.4mm_EP1.78x2.35mm, symbol grapto-v3w:MAX17260TFDN
- added C4: (no value), symbol Device:C
- added R29, R5: (no value), Resistor_SMD:R_0603_1608Metric_Pad0.98x0.95mm_HandSolder, symbol Device:R
- added TP25: TestPoint, TestPoint:TestPoint_THTPad_D2.0mm_Drill1.0mm, symbol Connector:TestPoint
- TP10, TP11, TP12: footprint (none) -> TestPoint:TestPoint_THTPad_D2.0mm_Drill1.0mm
- U8: value AP9211S-AL -> (none); footprint grapto-v3w:U-DFN2030-6_type_c -> (none)
- U9: value MCP7383x-2xMC -> (none); footprint Package_DFN_QFN:DFN-8-1EP_3x2mm_P0.5mm_EP1.75x1.45mm -> (none)
Connections:
- net p- is gone; now on net sysgnd: R16.2, U8.6 (S2)
- net low_batt: now also C4.1, R29.1, R5.2, TP25.1
- net p+: now also R5.1
- net sysgnd: now also C4.2, R29.2
- no-connect marks 2 -> 0
Other:
- note added: "1.67 V - 2.83 V"
- note added: "2.5 V - 4.25 V"
- note added: "Capacitor is used to provide current when adc is measuring"
- note added: "TODO - check how to schedule battery measuerments in ZMK - check accuracy of ADC at different impedances/currents - check leakage current of ADC pin - experiment with different values for resistor - experiment with different values for capacitor"

Commit message: Adjusting schematic to improve layout.
Parts:
- removed TP25: TestPoint, TestPoint:TestPoint_THTPad_D2.0mm_Drill1.0mm, symbol Connector:TestPoint
- C5: renamed from C4; value (none) -> .1u; footprint (none) -> Capacitor_SMD:C_0603_1608Metric_Pad1.08x0.95mm_HandSolder
- R19: renamed from R5; value (none) -> 1M
- R30: renamed from R29; value (none) -> 2M
- U8: value (none) -> AP9211S-AL; footprint (none) -> grapto-v3w:U-DFN2030-6_type_c
- U9: value (none) -> MCP7383x-2xMC; footprint (none) -> Package_DFN_QFN:DFN-8-1EP_3x2mm_P0.5mm_EP1.75x1.45mm
Changed lines of the file:
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@@
   (junction (at 110.49 72.39) (diameter 0) (color 0 0 0 0)
   )
-  (junction (at 100.33 126.365) (diameter 0) (color 0 0 0 0)
-  )
   (junction (at 228.6 60.96) (diameter 0) (color 0 0 0 0)
   )
@@
     (stroke (width 0) (type default) (color 0 0 0 0))
   )
-  (wire (pts (xy 88.9 126.365) (xy 100.33 126.365))
+  (wire (pts (xy 88.9 126.365) (xy 112.395 126.365))
     (stroke (width 0) (type default) (color 0 0 0 0))
   )
@@
   )
   (wire (pts (xy 188.595 83.185) (xy 188.595 86.36))
-    (stroke (width 0) (type default) (color 0 0 0 0))
-  )
-  (wire (pts (xy 100.33 126.365) (xy 112.395 126.365))
     (stroke (width 0) (type default) (color 0 0 0 0))
   )
@@
     )
     (property "Datasheet" "~" (id 3) (at 71.12 72.39 0)
-      (effects (font (size 1.27 1.27)) hide)
-    )
-    (pin "1")
-  )
-  (symbol (lib_id "Connector:TestPoint") (at 100.33 126.365 0) (unit 1)
-    (in_bom yes) (on_board yes) (fields_autoplaced)
-    (property "Reference" "TP25" (id 0) (at 101.727 122.2283 0)
-      (effects (font (size 1.27 1.27)) (justify left))
-    )
-    (property "Value" "TestPoint" (id 1) (at 101.727 124.7652 0)
-      (effects (font (size 1.27 1.27)) (justify left))
-    )
-    (property "Footprint" "TestPoint:TestPoint_THTPad_D2.0mm_Drill1.0mm" (id 2) (at 105.41 126.365 0)
-      (effects (font (size 1.27 1.27)) hide)
-    )
-    (property "Datasheet" "~" (id 3) (at 105.41 126.365 0)
       (effects (font (size 1.27 1.27)) hide)
     )
@@
     (in_bom yes) (on_board yes) (fields_autoplaced)
     (property "Reference" "U9" (id 0) (at 212.725 64.931 0))
-    (property "Value" "" (id 1) (at 212.725 67.4679 0))
-    (property "Footprint" "" (id 2) (at 212.725 81.28 0)
+    (property "Value" "MCP7383x-2xMC" (id 1) (at 212.725 67.4679 0))
+    (property "Footprint" "Package_DFN_QFN:DFN-8-1EP_3x2mm_P0.5mm_EP1.75x1.45mm" (id 2) (at 212.725 81.28 0)
       (effects (font (size 1.27 1.27)) hide)
     )
@@
   (symbol (lib_id "Device:R") (at 88.9 120.015 0) (unit 1)
     (in_bom yes) (on_board yes) (fields_autoplaced)
-    (property "Reference" "R5" (id 0) (at 90.678 119.1803 0)
-      (effects (font (size 1.27 1.27)) (justify left))
-    )
-    (property "Value" "" (id 1) (at 90.678 121.7172 0)
+    (property "Reference" "R19" (id 0) (at 90.678 119.1803 0)
+      (effects (font (size 1.27 1.27)) (justify left))
+    )
+    (property "Value" "1M" (id 1) (at 90.678 121.7172 0)
       (effects (font (size 1.27 1.27)) (justify left))
     )
@@
   (symbol (lib_id "Device:R") (at 88.9 134.62 0) (unit 1)
     (in_bom yes) (on_board yes) (fields_autoplaced)
-    (property "Reference" "R29" (id 0) (at 90.678 133.7853 0)
-      (effects (font (size 1.27 1.27)) (justify left))
-    )
-    (property "Value" "" (id 1) (at 90.678 136.3222 0)
+    (property "Reference" "R30" (id 0) (at 90.678 133.7853 0)
+      (effects (font (size 1.27 1.27)) (justify left))
+    )
+    (property "Value" "2M" (id 1) (at 90.678 136.3222 0)
       (effects (font (size 1.27 1.27)) (justify left))
     )
@@
     (in_bom yes) (on_board yes) (fields_autoplaced)
     (property "Reference" "U8" (id 0) (at 96.52 50.326 0))
-    (property "Value" "" (id 1) (at 96.52 52.8629 0))
-    (property "Footprint" "" (id 2) (at 100.33 66.675 0)
+    (property "Value" "AP9211S-AL" (id 1) (at 96.52 52.8629 0))
+    (property "Footprint" "grapto-v3w:U-DFN2030-6_type_c" (id 2) (at 100.33 66.675 0)
       (effects (font (size 1.27 1.27)) hide)
     )
@@
   (symbol (lib_id "Device:C") (at 77.47 134.62 0) (unit 1)
     (in_bom yes) (on_board yes) (fields_autoplaced)
-    (property "Reference" "C4" (id 0) (at 80.391 133.7853 0)
-      (effects (font (size 1.27 1.27)) (justify left))
-    )
-    (property "Value" "" (id 1) (at 80.391 136.3222 0)
-      (effects (font (size 1.27 1.27)) (justify left))
-    )
-    (property "Footprint" "" (id 2) (at 78.4352 138.43 0)
-      (effects (font (size 1.27 1.27)) hide)
-    )
+    (property "Reference" "C5" (id 0) (at 80.391 133.7853 0)
+      (effects (font (size 1.27 1.27)) (justify left))
+    )
+    (property "Value" ".1u" (id 1) (at 80.391 136.3222 0)
+      (effects (font (size 1.27 1.27)) (justify left))
+    )
+    (property "Footprint" "Capacitor_SMD:C_0603_1608Metric_Pad1.08x0.95mm_HandSolder" (id 2) (at 78.4352 138.43 0)
+      (effects (font (size 1.27 1.27)) hide)
+    )

Commit message: 2-layer layout ready to order.
Parts:
- TP10, TP11, TP12: footprint TestPoint:TestPoint_THTPad_D2.0mm_Drill1.0mm -> grapto-v3w:TestPoint_THTPad_D2.0mm_Drill1.0mm
Changed lines of the file:
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@@
       (effects (font (size 1.27 1.27)) (justify left))
     )
-    (property "Footprint" "TestPoint:TestPoint_THTPad_D2.0mm_Drill1.0mm" (id 2) (at 71.12 72.39 0)
+    (property "Footprint" "grapto-v3w:TestPoint_THTPad_D2.0mm_Drill1.0mm" (id 2) (at 71.12 72.39 0)
       (effects (font (size 1.27 1.27)) hide)
     )
@@
       (effects (font (size 1.27 1.27)) (justify left))
     )
-    (property "Footprint" "TestPoint:TestPoint_THTPad_D2.0mm_Drill1.0mm" (id 2) (at 59.69 45.72 0)
+    (property "Footprint" "grapto-v3w:TestPoint_THTPad_D2.0mm_Drill1.0mm" (id 2) (at 59.69 45.72 0)
       (effects (font (size 1.27 1.27)) hide)
     )
@@
       (effects (font (size 1.27 1.27)) (justify left))
     )
-    (property "Footprint" "TestPoint:TestPoint_THTPad_D2.0mm_Drill1.0mm" (id 2) (at 82.55 45.72 0)
+    (property "Footprint" "grapto-v3w:TestPoint_THTPad_D2.0mm_Drill1.0mm" (id 2) (at 82.55 45.72 0)
       (effects (font (size 1.27 1.27)) hide)
     )
