File: grapto-v3w-shared/matrix.kicad_sch (KiCad schematic)
At the start: 58 parts

Commit message: left half pcb draft.
Parts:
- D1, D10, D11, D12, D13, D14, D15, D16, D17, D18, D19, D2, D20, D21, D22, D23, D24, D25, D26, D27, D28, D29, D3, D4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: footprint Diode_SMD:D_SOD-123 -> (none)
