File: grapto-v3w-shared/battery_management.kicad_sch (KiCad schematic)
At the start: 15 parts, among them SW31 SW_SPDT, U4 BQ24075RGT

Commit message: Production files sent to jlcpcb.
Parts:
- R19: value 1M -> 1M2
- R30: value 2M -> 3M
Changed lines of the file:
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@@
       (effects (font (size 1.27 1.27)) (justify left))
     )
-    (property "Value" "1M" (at 70.993 114.0972 0)
+    (property "Value" "1M2" (at 70.993 114.0972 0)
       (effects (font (size 1.27 1.27)) (justify left))
     )
@@
   (symbol (lib_id "Device:R") (at 69.215 127 0) (unit 1)
     (in_bom yes) (on_board yes) (dnp no) (fields_autoplaced)
-    (property "Reference" "R30" (at 70.993 126.1653 0)
+    (property "Reference" "R30" (at 70.993 126.3563 0)
       (effects (font (size 1.27 1.27)) (justify left))
     )
-    (property "Value" "2M" (at 70.993 128.7022 0)
+    (property "Value" "3M" (at 70.993 128.2773 0)
       (effects (font (size 1.27 1.27)) (justify left))
     )
