File: grapto-v3w-shared/controller.kicad_sch (KiCad schematic)
At the start: 35 parts, among them J1 Conn_01x02_Female, J2 Conn_01x01_Female, J6 USB_C_Receptacle_USB2.0, J8 Conn_01x06_Male, U1 ACN52840, U2 TPS62822DLC, U3 USBLC6-2SC6

Commit message: Right pcb almost finished.
Parts:
- C16, C17, C2, C3, C4, C6, C7: footprint Fuse:Fuse_0603_1608Metric_Pad1.05x0.95mm_HandSolder -> Capacitor_SMD:C_0603_1608Metric_Pad1.08x0.95mm_HandSolder
- J2: footprint (none) -> TestPoint:TestPoint_THTPad_D2.0mm_Drill1.0mm
- J6: footprint Connector_USB:USB_C_Receptacle_G-Switch_GT-USB-7010ASV -> grapto-v3w:USB_C_Receptacle_molex_2169900001
- TP13, TP14, TP15, TP16, TP17, TP18, TP22: footprint Connector_PinHeader_2.54mm:PinHeader_1x01_P2.54mm_Vertical -> TestPoint:TestPoint_THTPad_D2.0mm_Drill1.0mm
Connections:
- net vusb: no longer U3.5 (VBUS)
- net vbus_fused: now reaches F4.2, R13.1, TP13.1
- net vbus_fused: now also U3.5 (VBUS)

Commit message: Production files sent to jlcpcb.
Parts:
- J6: footprint grapto-v3w:USB_C_Receptacle_molex_2169900001 -> grapto-v3w:USB_C_Receptacle_G-Switch_GT-USB-7004
- R1: value 62 -> 68
Changed lines of the file:
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@@
       (effects (font (size 1.27 1.27)))
     )
-    (property "Footprint" "grapto-v3w:USB_C_Receptacle_molex_2169900001" (at 43.815 154.94 0)
+    (property "Footprint" "grapto-v3w:USB_C_Receptacle_G-Switch_GT-USB-7004" (at 43.815 154.94 0)
       (effects (font (size 1.27 1.27)) hide)
     )
@@
       (effects (font (size 1.27 1.27)) (justify left))
     )
-    (property "Value" "62" (at 144.145 109.855 0)
-      (effects (font (size 1.27 1.27)) (justify left))
-    )
+    (property "Value" "68" (at 144.145 109.855 0)
+      (effects (font (size 1.27 1.27)) (justify left))
+    )
