File: grapto-v3w-right/grapto-v3w-right.kicad_pcb (KiCad board)
At the start: 2 copper layers, 150 x 124.7 mm, 59 parts

Commit message: update generated pcbs
Parts:
- moved USBC1 3.00 mm to (129.0, 93.8)
Other:
- board size 150 x 124.7 mm -> 150 x 127.7 mm

Commit message: left half pcb draft.
Parts:
- removed USBC1: TRRS-PJ-320A-dual, TRRS-PJ-320A-dual
- added C1: 1u, Capacitor_SMD:C_0603_1608Metric_Pad1.08x0.95mm_HandSolder, F.Cu at (168.9, 63.8)
- added C10: 22u, Fuse:Fuse_0603_1608Metric_Pad1.05x0.95mm_HandSolder, F.Cu at (168.9, 66.3)
- added C16: 22u, Fuse:Fuse_0603_1608Metric_Pad1.05x0.95mm_HandSolder, F.Cu at (148.1, 60.8)
- added C17: 22u, Fuse:Fuse_0603_1608Metric_Pad1.05x0.95mm_HandSolder, F.Cu at (142.2, 65.8)
- added C2: 120p, Fuse:Fuse_0603_1608Metric_Pad1.05x0.95mm_HandSolder, F.Cu at (137.8, 65.1)
- added C3: 22u, Fuse:Fuse_0603_1608Metric_Pad1.05x0.95mm_HandSolder, F.Cu at (133.5, 65.1)
- added C4: 22u, Fuse:Fuse_0603_1608Metric_Pad1.05x0.95mm_HandSolder, F.Cu at (142.2, 68.3)
- added C5: .1u, Capacitor_SMD:C_0603_1608Metric_Pad1.08x0.95mm_HandSolder, F.Cu at (173.5, 58.8)
- added C6: 22u, Fuse:Fuse_0603_1608Metric_Pad1.05x0.95mm_HandSolder, F.Cu at (133.5, 67.6)
- added C7: 22u, Fuse:Fuse_0603_1608Metric_Pad1.05x0.95mm_HandSolder, F.Cu at (148.9, 53.8)
- added D30, D59: , ComboDiode, F.Cu at (221.5, 184.5)
- added D31, D60: , ComboDiode, F.Cu at (221.5, 167.0)
- added D32, D61: , ComboDiode, F.Cu at (221.5, 149.5)
- added D33, D62: , ComboDiode, F.Cu at (203.0, 184.5)
- added D34, D63: , ComboDiode, F.Cu at (203.0, 167.0)
- added D35, D64: , ComboDiode, F.Cu at (203.0, 149.5)
- added D36, D65: , ComboDiode, F.Cu at (203.0, 132.0)
- added D37, D66: , ComboDiode, F.Cu at (184.5, 184.5)
- added D38, D67: , ComboDiode, F.Cu at (184.5, 167.0)
- added D39, D68: , ComboDiode, F.Cu at (184.5, 149.5)
- added D40, D69: , ComboDiode, F.Cu at (184.5, 132.0)
- added D41, D70: , ComboDiode, F.Cu at (184.5, 114.5)
- added D42, D71: , ComboDiode, F.Cu at (166.0, 179.5)
- added D43, D72: , ComboDiode, F.Cu at (166.0, 162.0)
- added D44, D73: , ComboDiode, F.Cu at (166.0, 144.5)
- added D45, D74: , ComboDiode, F.Cu at (166.0, 127.0)
- added D46, D75: , ComboDiode, F.Cu at (166.0, 109.5)
- added D47, D76: , ComboDiode, F.Cu at (147.5, 184.5)
- added D48, D77: , ComboDiode, F.Cu at (147.5, 167.0)
- added D49, D78: , ComboDiode, F.Cu at (147.5, 149.5)
- added D50, D79: , ComboDiode, F.Cu at (147.5, 132.0)
- added D51, D80: , ComboDiode, F.Cu at (147.5, 114.5)
- added D52, D81: , ComboDiode, F.Cu at (129.0, 171.0)
- added D53, D82: , ComboDiode, F.Cu at (129.0, 153.5)
- added D54, D83: , ComboDiode, F.Cu at (129.0, 136.0)
- added D55, D84: , ComboDiode, F.Cu at (129.0, 118.5)
- added D56, D85: , ComboDiode, F.Cu at (128.8, 191.6)
- added D57, D86: , ComboDiode, F.Cu at (109.7, 199.3)
- added D58, D87: , ComboDiode, F.Cu at (94.5, 213.2)
- added F3: Polyfuse, Fuse:Fuse_0603_1608Metric_Pad1.05x0.95mm_HandSolder, F.Cu at (174.2, 53.8)
- added F4: Polyfuse, Fuse:Fuse_0603_1608Metric_Pad1.05x0.95mm_HandSolder, F.Cu at (143.7, 58.3)
- added J1: Conn_01x02_Female, Connector_JST:JST_PH_S2B-PH-SM4-TB_1x02-1MP_P2.00mm_Horizontal, F.Cu at (136.4, 58.2)
- added J8: Conn_01x06_Male, Connector_PinHeader_2.54mm:PinHeader_1x06_P2.54mm_Vertical, F.Cu at (129.0, 54.9)
- added R1: 62, Resistor_SMD:R_0603_1608Metric_Pad0.98x0.95mm_HandSolder, F.Cu at (148.1, 58.3)
- added R13: 0.01m, Resistor_SMD:R_0603_1608Metric_Pad0.98x0.95mm_HandSolder, F.Cu at (143.7, 63.3)
- added R14: 0.01m, Resistor_SMD:R_0603_1608Metric_Pad0.98x0.95mm_HandSolder, F.Cu at (169.8, 53.8)
- added R19: 1M, Resistor_SMD:R_0603_1608Metric_Pad0.98x0.95mm_HandSolder, F.Cu at (164.5, 66.3)
- added R2: 0.01m, Resistor_SMD:R_0603_1608Metric_Pad0.98x0.95mm_HandSolder, F.Cu at (133.5, 70.1)
- added R20: 5.1k, Resistor_SMD:R_0603_1608Metric_Pad0.98x0.95mm_HandSolder, F.Cu at (137.8, 67.6)
- added R23: 5.1k, Resistor_SMD:R_0603_1608Metric_Pad0.98x0.95mm_HandSolder, F.Cu at (137.8, 70.1)
- added R24: 22, Resistor_SMD:R_0603_1608Metric_Pad0.98x0.95mm_HandSolder, F.Cu at (152.4, 56.3)
- added R25: 22, Resistor_SMD:R_0603_1608Metric_Pad0.98x0.95mm_HandSolder, F.Cu at (153.2, 53.8)
- added R30: 2M, Resistor_SMD:R_0603_1608Metric_Pad0.98x0.95mm_HandSolder, F.Cu at (174.2, 56.3)
- added R4: 10K, Resistor_SMD:R_0603_1608Metric_Pad0.98x0.95mm_HandSolder, F.Cu at (164.5, 63.8)
- added R5: 453k, Resistor_SMD:R_0603_1608Metric_Pad0.98x0.95mm_HandSolder, F.Cu at (152.4, 58.8)
- added R7: 3.3K, Resistor_SMD:R_0603_1608Metric_Pad0.98x0.95mm_HandSolder, F.Cu at (169.2, 59.1)
- added R8: 2.2K, Resistor_SMD:R_0603_1608Metric_Pad0.98x0.95mm_HandSolder, F.Cu at (169.8, 56.3)
- added R9: 100k, Resistor_SMD:R_0603_1608Metric_Pad0.98x0.95mm_HandSolder, F.Cu at (143.7, 60.8)
- added TP1: TestPoint, Connector_PinHeader_2.54mm:PinHeader_1x01_P2.54mm_Vertical, F.Cu at (164.7, 60.2)
- added U2: TPS62822DLC, Package_DFN_QFN:Texas_VSON-HR-8_1.5x2mm_P0.5mm, F.Cu at (157.3, 54.3)
- added U3: USBLC6-2SC6, Package_TO_SOT_SMD:SOT-23-6, F.Cu at (144.1, 54.8)
- added U4: BQ24075RGT, Package_DFN_QFN:VQFN-16-1EP_3x3mm_P0.5mm_EP1.6x1.6mm, F.Cu at (165.0, 55.2)
Connections:
- S30 pad 1: col5 -> col5row3
- S31 pad 1: col5 -> col5row2
- S32 pad 1: col5 -> col5row1
- S33 pad 1: col4 -> col4row3
- S34 pad 1: col4 -> col4row2
- S35 pad 1: col4 -> col4row1
- S36 pad 1: col4 -> col4row0
- S37 pad 1: col5 -> col5row4
- S38 pad 1: col3 -> col3row3
- S39 pad 1: col3 -> col3row2
- S40 pad 1: col3 -> col3row1
- S41 pad 1: col3 -> col3row0
- S42 pad 1: col4 -> col4row4
- S43 pad 1: col2 -> col2row3
- S44 pad 1: col2 -> col2row2
- S45 pad 1: col2 -> col2row1
- S46 pad 1: col2 -> col2row0
- S47 pad 1: col3 -> col3row4
- S48 pad 1: col1 -> col1row3
- S49 pad 1: col1 -> col1row2
- S50 pad 1: col1 -> col1row1
- S51 pad 1: col1 -> col1row0
- S52 pad 1: col0 -> col0row3
- S53 pad 1: col0 -> col0row2
- S54 pad 1: col0 -> col0row1
- S55 pad 1: col0 -> col0row0
- S56 pad 1: col2 -> col2row4
- S57 pad 1: col1 -> col1row4
- S58 pad 1: col0 -> col0row4
- S59 pad 1: col5 -> col5row3
- S60 pad 1: col5 -> col5row2
- S61 pad 1: col5 -> col5row1
- S62 pad 1: col4 -> col4row3
- S63 pad 1: col4 -> col4row2
- S64 pad 1: col4 -> col4row1
- S65 pad 1: col4 -> col4row0
- S66 pad 1: col5 -> col5row4
- S67 pad 1: col3 -> col3row3
- S68 pad 1: col3 -> col3row2
- S69 pad 1: col3 -> col3row1
- S70 pad 1: col3 -> col3row0
- S71 pad 1: col4 -> col4row4
- S72 pad 1: col2 -> col2row3
- S73 pad 1: col2 -> col2row2
- S74 pad 1: col2 -> col2row1
- S75 pad 1: col2 -> col2row0
- S76 pad 1: col3 -> col3row4
- S77 pad 1: col1 -> col1row3
- S78 pad 1: col1 -> col1row2
- S79 pad 1: col1 -> col1row1
- S80 pad 1: col1 -> col1row0
- S81 pad 1: col0 -> col0row3
- S82 pad 1: col0 -> col0row2
- S83 pad 1: col0 -> col0row1
- S84 pad 1: col0 -> col0row0
- S85 pad 1: col2 -> col2row4
- S86 pad 1: col1 -> col1row4
- S87 pad 1: col0 -> col0row4
Other:
- board size 150 x 127.7 mm -> 154.6 x 130.6 mm

Commit message: Right pcb almost finished.
Parts:
- added J2: Conn_01x01_Female, TestPoint:TestPoint_THTPad_D2.0mm_Drill1.0mm, F.Cu at (137.3, 98.7)
- added J6: USB_C_Receptacle_USB2.0, grapto-v3w:USB_C_Receptacle_molex_2169900001, B.Cu at (128.9, 94.1)
- added L2: 470n, grapto-v3w:MHCI05020-R47M-R8, B.Cu at (106.0, 156.9)
- added SW31: SW_SPDT, grapto-v3w:SW_SK-3296S-01-L2, B.Cu at (113.4, 118.4)
- added TP10: TestPoint, TestPoint:TestPoint_THTPad_D2.0mm_Drill1.0mm, F.Cu at (109.8, 140.1)
- added TP11: TestPoint, TestPoint:TestPoint_THTPad_D2.0mm_Drill1.0mm, F.Cu at (121.0, 126.3)
- added TP13: TestPoint, TestPoint:TestPoint_THTPad_D2.0mm_Drill1.0mm, F.Cu at (125.8, 111.9)
- added TP14: TestPoint, TestPoint:TestPoint_THTPad_D2.0mm_Drill1.0mm, F.Cu at (118.3, 111.0)
- added TP15: TestPoint, TestPoint:TestPoint_THTPad_D2.0mm_Drill1.0mm, F.Cu at (142.1, 98.5)
- added TP16: TestPoint, TestPoint:TestPoint_THTPad_D2.0mm_Drill1.0mm, F.Cu at (107.2, 145.3)
- added TP17: TestPoint, TestPoint:TestPoint_THTPad_D2.0mm_Drill1.0mm, F.Cu at (97.0, 158.8)
- added TP18: TestPoint, TestPoint:TestPoint_THTPad_D2.0mm_Drill1.0mm, F.Cu at (97.1, 163.4)
- added TP22: ~, TestPoint:TestPoint_THTPad_D2.0mm_Drill1.0mm, F.Cu at (118.4, 143.6)
- added U1: ACN52840, grapto-v3w:ACN52840, B.Cu at (108.6, 173.4)
- C1, C5, F3, F4, J1, J8, R1, R13, R14, R19, R2, R20, R23, R24, R25, R30, R4, R5, R7, R8, R9, U2, U3, U4: moved to B.Cu
- C10, C16, C17, C2, C3, C4, C6, C7: footprint Fuse:Fuse_0603_1608Metric_Pad1.05x0.95mm_HandSolder -> Capacitor_SMD:C_0603_1608Metric_Pad1.08x0.95mm_HandSolder; moved to B.Cu
- D30, D31, D32: value (none) -> LED_ARGB; footprint ComboDiode -> grapto-v3w:23-23B-R6GHBHC-A01-2A; moved to B.Cu
- TP1: footprint Connector_PinHeader_2.54mm:PinHeader_1x01_P2.54mm_Vertical -> TestPoint:TestPoint_THTPad_D2.0mm_Drill1.0mm; moved to B.Cu
- moved J8 153.1 mm to (110.8, 206.9), turned to -90 degrees
- moved C7 128.7 mm to (121.4, 179.6), turned to 180 degrees
- moved C3 125.8 mm to (100.2, 186.4), turned to 180 degrees
- moved C4 119.8 mm to (118.4, 185.8)
- moved D30 115.8 mm to (114.0, 141.5), turned to 180 degrees
- moved U2 109.0 mm to (108.2, 151.6), turned to -90 degrees
- moved D31 108.8 mm to (114.0, 150.5), turned to 180 degrees
- moved D32 108.0 mm to (114.0, 159.5), turned to 180 degrees
- moved R25 107.8 mm to (122.8, 157.2), turned to -90 degrees
- moved R30 107.0 mm to (117.0, 146.7), turned to 90 degrees
- moved C5 106.3 mm to (119.8, 150.6), turned to -90 degrees
- moved R5 105.1 mm to (103.0, 151.6), turned to 90 degrees
- moved R24 104.4 mm to (120.5, 155.8), turned to -90 degrees
- moved F3 103.9 mm to (111.0, 136.3), turned to 90 degrees
- moved R9 100.5 mm to (100.6, 151.6), turned to -90 degrees
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Connections:
- net /controller/vsys renamed vsys
- net Net-(R24-Pad1) renamed USB0_N
- net Net-(R25-Pad1) renamed USB0_P
- D30 pad 1: col5row3 -> /controller/vdd
- D30 pad 2: col5 -> Net-(D30-RK)
- D31 pad 1: col5row2 -> /controller/vdd
- D31 pad 2: col5 -> unconnected-(D31-RK-Pad2)
- D32 pad 1: col5row1 -> /controller/vdd
- D32 pad 2: col5 -> unconnected-(D32-RK-Pad2)
- F4 pad 2: Net-(F4-Pad2) -> vbus_fused
- R1 pad 2: Net-(D30-Pad2) -> Net-(D30-RK)
- R13 pad 1: Net-(F4-Pad2) -> vbus_fused
- U3 pad 5: /controller/vusb -> vbus_fused
Routing:
- net /controller/vdd: track 0.00 -> 144.4 mm, vias 0 -> 2
- net /controller/vusb: track 0.00 -> 142.3 mm
- net /controller/status1: track 0.00 -> 112.2 mm, vias 0 -> 4
- net /controller/swdio: track 0.00 -> 79.0 mm, vias 0 -> 4
- net /controller/fast_chg: track 0.00 -> 75.5 mm
- net /controller/swdclk: track 0.00 -> 70.2 mm, vias 0 -> 2
- net sysgnd: track 0.00 -> 65.5 mm, vias 0 -> 37
- net USB0_P: track 0.00 -> 61.1 mm
- net USB0_N: track 0.00 -> 59.6 mm
- net vsys: track 0.00 -> 50.3 mm
- net /controller/BatteryManagement/bat_fused: track 0.00 -> 44.9 mm
- net /controller/chg_led: track 0.00 -> 35.9 mm
- net USB_N: track 0.00 -> 34.8 mm
- net /controller/fast_chg_led: track 0.00 -> 31.7 mm
- net row4: track 0.00 -> 31.2 mm
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- added copper zone on F.Cu, net sysgnd
Other:
- board size 154.6 x 130.6 mm -> 154.6 x 129.3 mm

Commit message: Production files sent to jlcpcb.
Parts:
- J2, TP10, TP11, TP14, TP15, TP16, TP17, TP18, TP22: moved to B.Cu
- J6: footprint grapto-v3w:USB_C_Receptacle_molex_2169900001 -> grapto-v3w:USB_C_Receptacle_G-Switch_GT-USB-7004
- R1: value 62 -> 68
- R19: value 1M -> 1M2
- R30: value 2M -> 3M
- moved U3 5.02 mm to (138.8, 105.8)
- moved F4 4.91 mm to (122.4, 99.2)
- moved J6 3.41 mm to (129.1, 97.5)
- turned J2 to 180 degrees
- turned TP10 to 180 degrees
- turned TP11 to 180 degrees
- turned TP14 to 180 degrees
- turned TP15 to 180 degrees
- turned TP16 to 180 degrees
- turned TP17 to 180 degrees
- turned TP18 to 180 degrees
- turned TP22 to 180 degrees
Routing:
- net col4: track 0.00 -> 274.4 mm, vias 0 -> 6
- net col5: track 0.00 -> 270.9 mm, vias 0 -> 6
- net row0: track 0.00 -> 217.5 mm, vias 0 -> 12
- net row1: track 0.00 -> 207.6 mm, vias 0 -> 18
- net row2: track 0.00 -> 181.6 mm, vias 0 -> 20
- net row4: track 31.2 -> 197.7 mm, vias 0 -> 6
- net row3: track 0.00 -> 160.7 mm, vias 0 -> 18
- net col3: track 0.00 -> 151.8 mm
- net col0: track 0.00 -> 142.4 mm, vias 0 -> 12
- net col2: track 0.00 -> 141.4 mm, vias 0 -> 6
- net col1: track 0.00 -> 137.7 mm, vias 0 -> 10
- net col2row4: track 0.00 -> 11.4 mm
- net col0row4: track 0.00 -> 11.4 mm
- net col0row0: track 0.00 -> 11.4 mm
- net col1row0: track 0.00 -> 11.2 mm
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Other:
- outline, holes or cut-outs redrawn
- board text added: "+"
- board text added: "3.3V"
- board text added: "4.2 V Li ion >500 mAh"
- board text added: "D33"
- board text added: "Grapto-v3w rev2"
- board text added: "Herman Lundkvist 2023"
- board text added: "gnd"
- board text added: "right"
- board text added: "rst"
- board text added: "s30"
- board text added: "stat1"
- board text added: "swdclk"
- board text added: "swdio"
